File: design/r1.2/kicad/Glue.sch (KiCad schematic (older format))
At the start: 34 parts, among them IC2 ATF16V8BQL-15PU, IC3 ATF16V8BQL-15PU, IC5 ATF16V8BQL-15PU, IC6 74174N, IC7 74LS93, IC8 555N, IC9 74LS01N, Q2 5H8ET-10.000, Q3 5H8ET-4.000

Commit message: Update board for IC5 and tidy up
Parts:
- R21: value 4K7 -> 2K2
Connections:
- net A17: no longer IC5.11 (OE)
- net A19: now also IC5.11 (OE)
- net EXPSEL: now also IC5.15 (IO5)
- net MFPDS: now also IC5.12 (IO8); no longer IC5.15 (IO5)
- no-connect marks 12 -> 11
Changed lines of the file:
@@
 Text GLabel 10950 3200 2    47   Output ~ 0
 DTACK
-Text GLabel 10300 3600 2    47   Output ~ 0
+Text GLabel 10300 3900 2    47   Output ~ 0
 MFPDS
 Text GLabel 10300 3500 2    47   Output ~ 0
@@
 	1    0    0    -1
 $EndComp
-NoConn ~ 10300 3900
 $Comp
 L power:GND #PWR?
@@
 AR Path="/5E53B952/5F2C84D7" Ref="R21"  Part="1"
 F 0 "R21" V 10700 2759 59  0000 L BNN
-F 1 "4K7" V 10880 2750 59  0000 L BNN
+F 1 "2K2" V 10880 2750 59  0000 L BNN
 F 2 "rosco_m68k:0207_10" H 10850 2700 50  0001 C CNN
 F 3 "" H 10850 2700 50  0001 C CNN
@@
 	10300 3000 11350 3000
 Text Label 11200 3000 0    50   ~ 0
-A17
+A19
 Wire Wire Line
 	10300 3200 10850 3200
@@
 Wire Bus Line
 	19400 6050 19400 7500
+Text GLabel 10300 3600 2    50   Input ~ 0
+EXPSEL
 $EndSCHEMATC
