File: design/r2020/kicad/DUART.kicad_sch (KiCad schematic)
At the start: 17 parts, among them IC4 XR68C681CJTR-F, J1 UART_A, J2 UART_B, J4 Conn_01x06, J7 Conn_01x01_Male, Q1 3.6864MHz

Commit message: Feature/kicad 7 (#388)
* Update r2 to Kicad 7
* Update r2020 to Kicad 7
* Complete Kicad 7 migration
Parts:
- J1, J2: symbol Connector:Conn_01x06_Male -> Connector:Conn_01x06_Pin
- J7: symbol Connector:Conn_01x01_Male -> Connector:Conn_01x01_Pin
