File: design/r2020/kicad/Memory.kicad_sch (KiCad schematic)
At the start: 10 parts, among them U1 SST39SF040, U2 SST39SF040, U3 AS6C4008-55PCN, U4 AS6C4008-55PCN

Commit message: Complete Kicad 7 migration
Changed lines of the file:
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@@
     (comment 4 "Copyright 2019-2022 Ross Bamford and Contributors")
   )
-  (junction (at 25.4 92.71) (diameter 0) (color 0 0 0 0)
-  )
   (junction (at 115.57 30.48) (diameter 0) (color 0 0 0 0)
   )
+  (junction (at 25.4 119.38) (diameter 0) (color 0 0 0 0)
+  )
   (junction (at 201.93 30.48) (diameter 0) (color 0 0 0 0)
   )
-  (junction (at 25.4 186.69) (diameter 0) (color 0 0 0 0)
-  )
-  (junction (at 25.4 29.21) (diameter 0) (color 0 0 0 0)
+  (junction (at 25.4 96.52) (diameter 0) (color 0 0 0 0)
   )
   (junction (at 115.57 96.52) (diameter 0) (color 0 0 0 0)
   )
+  (junction (at 25.4 190.5) (diameter 0) (color 0 0 0 0)
+  )
   (junction (at 135.89 144.78) (diameter 0) (color 0 0 0 0)
   )
-  (junction (at 25.4 123.19) (diameter 0) (color 0 0 0 0)
+  (junction (at 25.4 25.4) (diameter 0) (color 0 0 0 0)
   )
   (junction (at 201.93 96.52) (diameter 0) (color 0 0 0 0)
   )
+  (wire (pts (xy 25.4 119.38) (xy 60.96 119.38))
+    (stroke (width 0) (type default))
+  )
+  (wire (pts (xy 25.4 190.5) (xy 25.4 192.405))
+    (stroke (width 0) (type default))
+  )
   (wire (pts (xy 220.98 96.52) (xy 201.93 96.52))
     (stroke (width 0) (type default))
   )
-  (wire (pts (xy 60.96 29.21) (xy 25.4 29.21))
-    (stroke (width 0) (type default))
-  )
-  (wire (pts (xy 25.4 92.71) (xy 25.4 95.25))
-    (stroke (width 0) (type default))
-  )
-  (wire (pts (xy 25.4 154.94) (xy 25.4 186.69))
+  (wire (pts (xy 25.4 60.96) (xy 25.4 96.52))
+    (stroke (width 0) (type default))
+  )
+  (wire (pts (xy 25.4 25.4) (xy 60.96 25.4))
+    (stroke (width 0) (type default))
+  )
+  (wire (pts (xy 60.96 96.52) (xy 25.4 96.52))
     (stroke (width 0) (type default))
   )
@@
     (stroke (width 0) (type default))
   )
-  (wire (pts (xy 60.96 123.19) (xy 25.4 123.19))
-    (stroke (width 0) (type default))
-  )
   (wire (pts (xy 115.57 22.86) (xy 115.57 30.48))
     (stroke (width 0) (type default))
   )
+  (wire (pts (xy 25.4 119.38) (xy 25.4 147.32))
+    (stroke (width 0) (type default))
+  )
   (wire (pts (xy 135.89 120.65) (xy 135.89 125.73))
     (stroke (width 0) (type default))
@@
     (stroke (width 0) (type default))
   )
-  (wire (pts (xy 60.96 186.69) (xy 25.4 186.69))
-    (stroke (width 0) (type default))
-  )
-  (wire (pts (xy 60.96 92.71) (xy 25.4 92.71))
-    (stroke (width 0) (type default))
-  )
   (wire (pts (xy 115.57 62.23) (xy 115.57 96.52))
     (stroke (width 0) (type default))
   )
-  (wire (pts (xy 25.4 123.19) (xy 25.4 115.57))
-    (stroke (width 0) (type default))
-  )
   (wire (pts (xy 134.62 96.52) (xy 115.57 96.52))
     (stroke (width 0) (type default))
@@
     (stroke (width 0) (type default))
   )
-  (wire (pts (xy 25.4 29.21) (xy 25.4 21.59))
-    (stroke (width 0) (type default))
-  )
   (wire (pts (xy 134.62 30.48) (xy 115.57 30.48))
     (stroke (width 0) (type default))
@@
     (stroke (width 0) (type default))
   )
-  (wire (pts (xy 25.4 60.96) (xy 25.4 92.71))
+  (wire (pts (xy 60.96 190.5) (xy 25.4 190.5))
     (stroke (width 0) (type default))
   )
@@
     (stroke (width 0) (type default))
   )
+  (wire (pts (xy 25.4 96.52) (xy 25.4 100.965))
+    (stroke (width 0) (type default))
+  )
+  (wire (pts (xy 25.4 25.4) (xy 25.4 53.34))
+    (stroke (width 0) (type default))
+  )
   (wire (pts (xy 106.68 144.78) (xy 116.84 144.78))
     (stroke (width 0) (type default))
   )
-  (wire (pts (xy 25.4 186.69) (xy 25.4 189.23))
-    (stroke (width 0) (type default))
-  )
-  (wire (pts (xy 25.4 123.19) (xy 25.4 147.32))
+  (wire (pts (xy 25.4 154.94) (xy 25.4 190.5))
+    (stroke (width 0) (type default))
+  )
+  (wire (pts (xy 25.4 115.57) (xy 25.4 119.38))
     (stroke (width 0) (type default))
   )
@@
     (stroke (width 0) (type default))
   )
-  (wire (pts (xy 25.4 29.21) (xy 25.4 53.34))
+  (wire (pts (xy 25.4 21.59) (xy 25.4 25.4))
     (stroke (width 0) (type default))
   )
@@
   (symbol (lib_id "Memory_Flash:SST39SF040") (at 60.96 62.23 0) (unit 1)
     (in_bom yes) (on_board yes) (dnp no)
-    (property "Reference" "U1" (at 60.96 26.4668 0)
+    (property "Reference" "U1" (at 60.96 19.177 0)
       (effects (font (size 1.7526 1.7526)))
     )
-    (property "Value" "SST39SF040" (at 60.96 29.5148 0)
+    (property "Value" "SST39SF040" (at 60.96 22.225 0)
       (effects (font (size 1.7526 1.7526)))
     )
@@
       (effects (font (size 1.27 1.27)) hide)
     )
-    (property "Datasheet" "" (at 60.96 62.23 0)
+    (property "Datasheet" "http://ww1.microchip.com/downloads/en/DeviceDoc/25022B.pdf" (at 60.96 62.23 0)
       (effects (font (size 1.27 1.27)) hide)
     )
@@
   (symbol (lib_id "Memory_Flash:SST39SF040") (at 60.96 156.21 0) (unit 1)
     (in_bom yes) (on_board yes) (dnp no)
-    (property "Reference" "U2" (at 60.96 120.4468 0)
+    (property "Reference" "U2" (at 60.96 113.03 0)
       (effects (font (size 1.7526 1.7526)))
     )
-    (property "Value" "SST39SF040" (at 60.96 123.4948 0)
+    (property "Value" "SST39SF040" (at 60.96 116.078 0)
       (effects (font (size 1.7526 1.7526)))
     )
@@
       (effects (font (size 1.27 1.27)) hide)
     )
-    (property "Datasheet" "" (at 60.96 156.21 0)
+    (property "Datasheet" "http://ww1.microchip.com/downloads/en/DeviceDoc/25022B.pdf" (at 60.96 156.21 0)
       (effects (font (size 1.27 1.27)) hide)
     )
@@
     )
   )
-  (symbol (lib_id "power:GND") (at 25.4 95.25 0) (unit 1)
+  (symbol (lib_id "power:GND") (at 25.4 100.965 0) (unit 1)
     (in_bom yes) (on_board yes) (dnp no)
-    (property "Reference" "#PWR0104" (at 25.4 101.6 0)
-      (effects (font (size 1.27 1.27)) hide)
-    )
-    (property "Value" "GND" (at 25.527 99.6442 0)
+    (property "Reference" "#PWR0104" (at 25.4 107.315 0)
+      (effects (font (size 1.27 1.27)) hide)
+    )
+    (property "Value" "GND" (at 25.527 105.3592 0)
       (effects (font (size 1.27 1.27)))
     )
-    (property "Footprint" "" (at 25.4 95.25 0)
-      (effects (font (size 1.27 1.27)) hide)
-    )
-    (property "Datasheet" "" (at 25.4 95.25 0)
+    (property "Footprint" "" (at 25.4 100.965 0)
+      (effects (font (size 1.27 1.27)) hide)
+    )
+    (property "Datasheet" "" (at 25.4 100.965 0)
       (effects (font (size 1.27 1.27)) hide)
     )
@@
     )
   )
-  (symbol (lib_id "power:GND") (at 25.4 189.23 0) (unit 1)
+  (symbol (lib_id "power:GND") (at 25.4 192.405 0) (unit 1)
     (in_bom yes) (on_board yes) (dnp no)
-    (property "Reference" "#PWR0106" (at 25.4 195.58 0)
-      (effects (font (size 1.27 1.27)) hide)
-    )
-    (property "Value" "GND" (at 25.527 193.6242 0)
+    (property "Reference" "#PWR0106" (at 25.4 198.755 0)
+      (effects (font (size 1.27 1.27)) hide)
+    )
+    (property "Value" "GND" (at 25.527 196.7992 0)
       (effects (font (size 1.27 1.27)))
     )
-    (property "Footprint" "" (at 25.4 189.23 0)
-      (effects (font (size 1.27 1.27)) hide)
-    )
-    (property "Datasheet" "" (at 25.4 189.23 0)
-      (effects (font (size 1.27 1.27)) hide)
-    )
+    (property "Footprint" "" (at 25.4 192.405 0)
+      (effects (font (size 1.27 1.27)) hide)
+    )
+    (property "Datasheet" "" (at 25.4 192.405 0)
+      (effects (font (size 1.27 1.27)) hide)
+    )
