File: design/r2/kicad/Memory.kicad_sch (KiCad schematic)
At the start: 10 parts, among them U1 SST39SF040, U2 SST39SF040, U3 AS6C4008-55PCN, U4 AS6C4008-55PCN

Commit message: Tentative r2 SMD design
Parts:
- C3, C4, C5, C6: footprint rosco_m68k:C2.5-3 -> Capacitor_SMD:C_0603_1608Metric
- R11: footprint rosco_m68k:0207_10 -> Resistor_SMD:R_0603_1608Metric
Changed lines of the file:
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@@
       (effects (font (size 1.27 1.27)) (justify left))
     )
-    (property "Footprint" "rosco_m68k:0207_10" (at 134.112 129.54 90)
+    (property "Footprint" "Resistor_SMD:R_0603_1608Metric" (at 134.112 129.54 90)
       (effects (font (size 1.27 1.27)) hide)
     )
@@
       (effects (font (size 1.4986 1.4986)) (justify left bottom))
     )
-    (property "Footprint" "rosco_m68k:C2.5-3" (at 25.4 149.86 0)
+    (property "Footprint" "Capacitor_SMD:C_0603_1608Metric" (at 25.4 149.86 0)
       (effects (font (size 1.27 1.27)) hide)
     )
@@
       (effects (font (size 1.4986 1.4986)) (justify left bottom))
     )
-    (property "Footprint" "rosco_m68k:C2.5-3" (at 115.57 57.15 0)
+    (property "Footprint" "Capacitor_SMD:C_0603_1608Metric" (at 115.57 57.15 0)
       (effects (font (size 1.27 1.27)) hide)
     )
@@
       (effects (font (size 1.4986 1.4986)) (justify left bottom))
     )
-    (property "Footprint" "rosco_m68k:C2.5-3" (at 201.93 57.15 0)
+    (property "Footprint" "Capacitor_SMD:C_0603_1608Metric" (at 201.93 57.15 0)
       (effects (font (size 1.27 1.27)) hide)
     )
@@
       (effects (font (size 1.4986 1.4986)) (justify left bottom))
     )
-    (property "Footprint" "rosco_m68k:C2.5-3" (at 25.4 55.88 0)
-      (effects (font (size 1.27 1.27)) hide)
-    )
+    (property "Footprint" "Capacitor_SMD:C_0603_1608Metric" (at 25.4 55.88 0)
+      (effects (font (size 1.27 1.27)) hide)
+    )
