File: design/r2/kicad/CPU.kicad_sch (KiCad schematic)
At the start: 8 parts, among them IC1 MC68010P10, Q2 5H8ET-10.000

Commit message: Feature/smd birdseed (#427)
* GAL changes to better support coprocessor

* Update designs for copro GAL change

* Revert accidental DUARTSEL changes

* Re-add mistakenly-removed polarity symbols

* Tentative r2 SMD design

* Resize tiny resistors

* More address lines into GALs

* Reroute for FTDI

* prod

* Correct FT2232HL part number

* Mask expansion and silk tidy after first spin
Parts:
- C7, C8: footprint rosco_m68k:C2.5-3 -> Capacitor_SMD:C_0603_1608Metric
- R10, R3, R7, R9: footprint rosco_m68k:0207_10 -> Resistor_SMD:R_0603_1608Metric
Changed lines of the file:
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@@
   (title_block
     (title "ROSCO_M68K GENERAL PURPOSE MC68010 COMPUTER")
-    (date "2024-03-09")
+    (date "2024-04-15")
     (rev "2.2")
     (company "The Really Old-School Company Limited")
@@
       (effects (font (size 1.4986 1.4986)) (justify left bottom))
     )
-    (property "Footprint" "rosco_m68k:0207_10" (at 193.04 121.92 0)
+    (property "Footprint" "Resistor_SMD:R_0603_1608Metric" (at 193.04 121.92 0)
       (effects (font (size 1.27 1.27)) hide)
     )
@@
       (effects (font (size 1.4986 1.4986)) (justify left bottom))
     )
-    (property "Footprint" "rosco_m68k:0207_10" (at 203.2 121.92 0)
+    (property "Footprint" "Resistor_SMD:R_0603_1608Metric" (at 203.2 121.92 0)
       (effects (font (size 1.27 1.27)) hide)
     )
@@
       (effects (font (size 1.4986 1.4986)) (justify left bottom))
     )
-    (property "Footprint" "rosco_m68k:0207_10" (at 213.36 121.92 0)
+    (property "Footprint" "Resistor_SMD:R_0603_1608Metric" (at 213.36 121.92 0)
       (effects (font (size 1.27 1.27)) hide)
     )
@@
       (effects (font (size 1.4986 1.4986)) (justify left bottom))
     )
-    (property "Footprint" "rosco_m68k:C2.5-3" (at 165.1 58.42 0)
+    (property "Footprint" "Capacitor_SMD:C_0603_1608Metric" (at 165.1 58.42 0)
       (effects (font (size 1.27 1.27)) hide)
     )
@@
       (effects (font (size 1.4986 1.4986)) (justify left bottom))
     )
-    (property "Footprint" "rosco_m68k:C2.5-3" (at 207.01 58.42 0)
+    (property "Footprint" "Capacitor_SMD:C_0603_1608Metric" (at 207.01 58.42 0)
       (effects (font (size 1.27 1.27)) hide)
     )
@@
       (effects (font (size 1.27 1.27)) (justify left))
     )
-    (property "Footprint" "rosco_m68k:0207_10" (at 172.212 48.26 90)
-      (effects (font (size 1.27 1.27)) hide)
-    )
+    (property "Footprint" "Resistor_SMD:R_0603_1608Metric" (at 172.212 48.26 90)
+      (effects (font (size 1.27 1.27)) hide)
+    )
