File: design/r2/kicad/Expansion.kicad_sch (KiCad schematic)
At the start: 33 parts, among them IC1 MC68010P10, IC13 TPS22929D, IC7 74LS148, J10 USB_C_Receptacle_PowerOnly_6P, J3 Conn_02x32_Odd_Even, J5 PWR, J6 Conn_01x05_Male, J9 Jack-DC

Commit message: prod
Parts:
- IC13: LCSC (none) -> 415177
Changed lines of the file:
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@@
+      (effects (font (size 1.27 1.27)) hide)
+    )
+    (property "LCSC" "415177" (at 137.16 78.74 0)
       (effects (font (size 1.27 1.27)) hide)
     )

Commit message: Mask expansion and silk tidy after first spin
Parts:
- IC13: LCSC 415177 -> C415177
Changed lines of the file:
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@@
   (title_block
     (title "ROSCO_M68K GENERAL PURPOSE MC68010 COMPUTER")
-    (date "2024-04-03")
+    (date "2024-04-15")
     (rev "2.2")
     (company "The Really Old-School Company Limited")
@@
       (effects (font (size 1.27 1.27)) hide)
     )
-    (property "LCSC" "415177" (at 137.16 78.74 0)
-      (effects (font (size 1.27 1.27)) hide)
-    )
+    (property "LCSC" "C415177" (at 137.16 78.74 0)
+      (effects (font (size 1.27 1.27)) hide)
+    )
