File: design/r2/kicad/FTDI.kicad_sch (KiCad schematic)
At the start: 38 parts, among them IC10 SN74LVC2G17, IC11 SN74LVC2G17, IC8 SN74LVC2G17, IC9 SN74LVC2G17, U1 93LC56BT-I/OT, U6 AP2127K-3.3, U6 FT2232HL, Y2 12MHz

Commit message: prod
Parts:
- FB1: LCSC (none) -> C82155
Changed lines of the file:
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@@
+      (effects (font (size 1.27 1.27)) hide)
+    )
+    (property "LCSC" "C82155" (at 248.92 20.32 90)
       (effects (font (size 1.27 1.27)) hide)
     )

Commit message: Mask expansion and silk tidy after first spin
Parts:
- C19: LCSC (none) -> C376778
- U6: LCSC C193662 -> C27882
Changed lines of the file:
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@@
   (title_block
     (title "ROSCO_M68K GENERAL PURPOSE MC68010 COMPUTER")
-    (date "2024-04-03")
+    (date "2024-04-15")
     (rev "2.2")
     (company "The Really Old-School Company Limited")
@@
       (effects (font (size 1.27 1.27)) hide)
     )
+    (property "LCSC" "C376778" (at 151.13 148.59 0)
+      (effects (font (size 1.27 1.27)) hide)
+    )
+    (property "Field5" "" (at 151.13 148.59 0)
+      (effects (font (size 1.27 1.27)) hide)
+    )
     (pin "1")
     (pin "2")
@@
       (effects (font (size 1.27 1.27)) hide)
     )
+    (property "LCSC" "C376778" (at 140.97 148.59 0)
+      (effects (font (size 1.27 1.27)) hide)
+    )
+    (property "Field5" "" (at 140.97 148.59 0)
+      (effects (font (size 1.27 1.27)) hide)
+    )
     (pin "1")
     (pin "2")
@@
       (effects (font (size 1.27 1.27)) hide)
     )
-    (property "LCSC" "C193662" (at 189.23 101.6 0)
-      (effects (font (size 1.27 1.27)) hide)
-    )
+    (property "LCSC" "C27882" (at 189.23 101.6 0)
+      (effects (font (size 1.27 1.27)) hide)
+    )

Commit message: Re-do initial r2.3 work
Parts:
- added JP5, JP6, JP7, JP8: Jumper_2_Small_Bridged, Jumper:SolderJumper-2_P1.3mm_Bridged_RoundedPad1.0x1.5mm, symbol Jumper:Jumper_2_Small_Bridged
- renumbered U6 to IC12, LED3 to LED5, LED3 to LED6, LED3 to LED7, LED3 to LED8, R13 to R20, R13 to R22, R13 to R23, R13 to R30, R13 to R33, R13 to R6
Connections:
- net CTSA: now also JP5.2 (B); no longer IC8.6 (Y1)
- net CTSB: now also JP8.2 (B); no longer IC10.4 (Y2)
- net RXDA: now also JP6.2 (B); no longer IC8.4 (Y2)
- net RXDB: now also JP7.2 (B); no longer IC10.6 (Y1)
- new net: IC10.4 (Y2), JP8.1 (A)
- new net: IC8.6 (Y1), JP5.1 (A)
- new net: IC10.6 (Y1), JP7.1 (A)
- new net: IC8.4 (Y2), JP6.1 (A)
Other:
- moved on the sheet: IC11, IC9
